File: Hardware/MTR_Charger_X5S.kicad_sch (KiCad schematic)
At the start: 46 parts, among them J1 Korean Hroparts Elec TYPE-C-3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, Q1 IRF7324TRPBF, U1 RP2040, U2 STUSB4500QTR, U3 ESDA25W, U4 LMV358IDR, U5 W25Q16JVUXIQ, X1 X322512MSB4SI

Commit message: RP2040 and QSPI Flash done
Parts:
- removed U4: LMV358IDR, easyeda2kicad:SOIC-8_L4.9-W3.9-P1.27-LS6.0-BL, symbol easyeda2kicad:LMV358IDR
- added BAT1, BAT2: BH-18650-B5BA016, easyeda2kicad:BAT-SMD_BH-18650-B5BA016, symbol easyeda2kicad:BH-18650-B5BA016
- added C21, C22: 1uF, symbol Device:C_Small
- added C23: 100nF, symbol Device:C_Small
- added J2: Micro_SD_Card, easyeda2kicad:TF-SMD_TF-04A, symbol Connector:Micro_SD_Card
- added JP1, JP2, JP3, JP4, JP5: SolderJumper_2_Bridged, Jumper:SolderJumper-2_P1.3mm_Bridged_Pad1.0x1.5mm, symbol Jumper:SolderJumper_2_Bridged
- added R15, R16, R17, R18: 4.7k, symbol Device:R_Small
- added R19, R28, R33, R38, R43: 33m, Resistor_SMD:R_2512_6332Metric, symbol Device:R
- added R20, R21, R27, R29, R32, R34, R37, R39, R42, R44: 1k, Resistor_SMD:R_0603_1608Metric, symbol Device:R_Small
- added R22, R23, R25, R26, R30, R31, R35, R36, R40, R41, R45: 100k, Resistor_SMD:R_0603_1608Metric, symbol Device:R_Small
- added R24: 27.4k, symbol Device:R_Small
- added SW1: Boot, easyeda2kicad:SW-SMD_L4.0-W3.0-LS5.0, symbol Switch:SW_Push
- added SW2: Reset, easyeda2kicad:SW-SMD_L4.0-W3.0-LS5.0, symbol Switch:SW_Push
- added U10, U11, U7, U8, U9: LMC6482AIMX/NOPB, easyeda2kicad:SOIC-8_L4.9-W3.9-P1.27-LS6.0-BL, symbol dk_Linear-Amplifiers-Instrumentation-OP-Amps-Buffer-Amps:LMV358IDR
- added U4, U6: LMV358IDR, digikey-footprints:SOIC-8_W3.9mm, symbol dk_Linear-Amplifiers-Instrumentation-OP-Amps-Buffer-Amps:LMV358IDR
Connections:
- net +3.3V: now also U5.8 (VCC), C22.1, C23.1, R16.2, R18.2
- net GND: now also U1.19 (TESTEN), U5.4 (GND), C21.1, C22.2, C23.2, R23.2, R26.2, R31.2, R36.2, R41.2, SW1.1, SW2.1, U10.4 (GND), U11.4 (GND), U7.4 (GND), U7.4 (GND), U8.4 (GND), U9.4 (GND)
- net SCL: now also U1.7 (GPIO5)
- net SDA: now also U1.6 (GPIO4)
- net QSPI_SS: now reaches U5.1 (~{CS})
- net QSPI_SS: now also U1.56 (QSPI_SS), R17.2, R18.1
- net QSPI_SD1: now reaches U5.2 (DO(IO1))
- net QSPI_SD1: now also U1.55 (QSPI_SD1)
- net QSPI_SD2: now reaches U5.3 (WP#(IO2))
- net QSPI_SD2: now also U1.54 (QSPI_SD2)
- net QSPI_SD0: now reaches U5.5 (DI(IO0))
- net QSPI_SD0: now also U1.53 (QSPI_SD0)
- net QSPI_CLK: now reaches U5.6 (CLK)
- net QSPI_CLK: now also U1.52 (QSPI_SCLK)
- net QSPI_SD3: now reaches U5.7 (RESET#(IO3))
- net QSPI_SD3: now also U1.51 (QSPI_SD3)
- net RUN: now reaches U1.26 (RUN)
- net RUN: now also C21.2, R15.2, R16.1
- new net: R17.1, SW1.2
- new net: R39.2, R40.1, U10.2
- new net: R26.1, R27.2, U8.3
- new net: R21.2, R22.1, U7.2
- new net: R22.2, U7.1
- new net: R15.1, SW2.2
- new net: R40.2, U10.1
- new net: R36.1, R37.2, U10.3
- new net: R41.1, R42.2, U11.3
- new net: U7.6, U7.7
- new net: R20.2, R23.1, U7.3
- new net: R29.2, R30.1, U8.2
- new net: R30.2, U8.1
- new net: R44.2, R45.1, U11.2
- new net: R31.1, R32.2, U9.3
- new net: R45.2, U11.1
- new net: R34.2, R35.1, U9.2
- new net: R35.2, U9.1
- new net +5V: U10.8 (VCC+), U11.8 (VCC+), U7.8 (VCC+), U7.8 (VCC+), U8.8 (VCC+), U9.8 (VCC+)
- new net CELL_01: BAT1.2, JP1.2 (B)
- new net CELL_02: BAT1.4, JP2.2 (B)
- new net CELL_03: BAT1.6, JP3.2 (B)
- new net CELL_04: BAT2.2, JP4.2 (B)
- new net CELL_05: BAT2.4, JP5.2 (B)
- new net sence_01+: R19.1, R20.1
- new net sence_01-: JP1.1 (A), R19.2, R21.1
- new net sence_02+: R27.1, R28.1
- new net sence_02-: JP2.1 (A), R28.2, R29.1
- new net sence_03+: R32.1, R33.1
- new net sence_03-: JP3.1 (A), R33.2, R34.1
- new net sence_04+: R37.1, R38.1
- new net sence_04-: JP4.1 (A), R38.2, R39.1
- new net sence_05+: R42.1, R43.1
- new net sence_05-: JP5.1 (A), R43.2, R44.1
- no-connect marks 7 -> 8
Other:
- added sheet Auto Power Switch Circuit (Auto_Power_Switch_Circuit.kicad_sch)
- added sheet Periodic battery level measurement simulation (Periodic_battery_level_measurement_simulation.kicad_sch)
- note added: "16MB QSPI Flash"
- note added: "Close to pin 45"
- note added: "Force flash storage boot"
- note added: "µC RP2040"
- moved on the sheet: C10, C11, C12, C13, C14, C15, C16, C17, C18, C19, C20, C8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
