File: Hardware/MTR_Charger_X5S.kicad_sch (KiCad schematic)
At the start: 65 parts, among them J1 Korean Hroparts Elec TYPE-C-3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, J2 Micro_SD_Card, Q1 IRF7324TRPBF, SW1 Boot, SW2 Reset, U1 W25Q16JVUXIQ, U2 RP2040, U3 ADS7830IPWR, U4 ADS7830IPWR, U5 ESDA25W, U6 STUSB4500QTR, U7 MCP73833-AMI/MF, U8 LMV358IDR, X1 X322512MSB4SI

Commit message: Add Mux for Battery charging current selection
Parts:
- added C25: 1uF, Capacitor_SMD:C_1206_3216Metric, symbol Device:C_Small
- added C26, C27: 1uF, symbol Device:C_Small
- added R100, R101, R102, R103, R99: 100R, symbol Device:R_Small
- added R104, R105, R106, R107, R108, R98: 1k, symbol Device:R_Small
- added R109, R110, R111, R112, R113, R114, R115, R116, R117, R118, R119, R120: 100k, symbol Device:R_Small
- added R97: NCP18XH103F03RB, easyeda2kicad:R0603, symbol easyeda2kicad:NCP18XH103F03RB
- added U14: TCA9535PWR_C130204, easyeda2kicad:TSSOP-24_L7.8-W4.4-P0.65-LS6.4-BL, symbol easyeda2kicad:TCA9535PWR_C130204
- added U15: CD74HCT4051M96, easyeda2kicad:SOP-16_L10.0-W3.9-P1.27-LS6.0-BL, symbol easyeda2kicad:CD74HCT4051M96_C406862
- C24: value 100nF -> 1uF
- D3: footprint Diode_SMD:D_0402_1005Metric -> easyeda2kicad:X2-DFN1006-2_L1.0-W0.6-P0.65-RD
- R11, R12: now not fitted; now left out of the parts list
- U8: footprint digikey-footprints:SOIC-8_W3.9mm -> easyeda2kicad:SOIC-8_L4.9-W3.9-P1.27-LS6.0-BL; LCSC (none) -> C63813
- U8: footprint digikey-footprints:SOIC-8_W3.9mm -> easyeda2kicad:SOIC-8_L4.9-W3.9-P1.27-LS6.0-BL
Connections:
- net +3.3V: now also R111.1, R112.1, R113.1, R114.1, R119.1, R120.1, U15.16 (VCC)
- net GND: now also C24.2, U3.11 (COM), U3.9 (GND), U4.11 (COM), U4.9 (GND), C25.2, C26.2, C27.2, R104.1, R109.1, R110.1, R97.1, R98.1, U14.12 (GND), U15.6 (~{E}), U15.7 (VEE), U15.8 (GND)
- net Vsnk: now also C24.1, U7.1 (VDD), U7.2 (VDD)
- net CHARGING_01: now reaches U7.10 (VBAT)
- net CHARGING_01: now also U7.9 (VBAT), C25.1
- net STAT1_Cell_01: now reaches U7.3 (STAT1)
- net STAT1_Cell_01: now also U14.6 (P02)
- net STAT2_Cell_01: now reaches U7.4 (STAT2)
- net STAT2_Cell_01: now also U14.5 (P01)
- net PROG_CELL_01: now reaches U7.6 (PROG)
- net PROG_CELL_01: now also U15.3 (A)
- net PG_Cell_01: now reaches U7.7 (~{PG})
- net PG_Cell_01: now also U14.4 (P00)
- net at U7.8 (THERM): now also R97.2
- net at U4.10 (REFIN/REFOUT): now also C26.1
- net at U4.12 (A0): now also R117.2, R120.2
- net at U4.13 (A1): now also R118.2, R119.2
- net at U3.10 (REFIN/REFOUT): now also C27.1
- net at U3.12 (A0): now also R114.2, R115.2
- net at U3.13 (A1): now also R113.2, R116.2
- new net: R100.1, R99.2, U15.14 (A1)
- new net: R100.2, R101.1, U15.15 (A2)
- new net: R109.2, R112.2, U14.3 (A2)
- new net: R98.2, R99.1, U15.13 (A0)
- new net: R104.2, R105.2
- new net: R117.1, R118.1
- new net: R103.2, U15.1 (A4)
- new net: R101.2, R102.1, U15.12 (A3)
- new net: R105.1, R106.2, U15.2 (A6)
- new net: R108.2, U15.4 (A7)
- new net: R106.1, R107.1, U15.5 (A5)
- new net: R115.1, R116.1
- new net: R107.2, R108.1
- new net: R110.2, R111.2, U14.2 (A1)
- new net: R102.2, R103.1
- new net Mux_CELL_01_S0: U14.9 (P05), U15.11 (S0)
- new net Mux_CELL_01_S1: U14.8 (P04), U15.10 (S1)
- new net Mux_CELL_01_S2: U14.7 (P03), U15.9 (S2)
Other:
- moved on the sheet: C24

Commit message: --------------
Other:
- moved on the sheet: J2
Changed lines of the file:
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@@
 	(symbol
 		(lib_id "Connector:Micro_SD_Card")
-		(at 643.89 99.06 0)
+		(at 589.28 87.63 0)
 		(unit 1)
 		(exclude_from_sim no)
@@
 		(fields_autoplaced yes)
 		(property "Reference" "J2"
-			(at 644.525 80.01 0)
+			(at 589.915 68.58 0)
 			(effects
 				(font
@@
 		)
 		(property "Value" "Micro_SD_Card"
-			(at 644.525 82.55 0)
+			(at 589.915 71.12 0)
 			(effects
 				(font
@@
 		)
 		(property "Footprint" "easyeda2kicad:TF-SMD_TF-04A"
-			(at 673.1 91.44 0)
+			(at 618.49 80.01 0)
 			(effects
 				(font
@@
 		)
 		(property "Datasheet" "http://katalog.we-online.de/em/datasheet/693072010801.pdf"
-			(at 643.89 99.06 0)
+			(at 589.28 87.63 0)
 			(effects
 				(font
@@
 		)
 		(property "Description" "Micro SD Card Socket"
-			(at 643.89 99.06 0)
+			(at 589.28 87.63 0)
 			(effects
 				(font
@@
 		)
 		(property "LCSC" "C145799"
-			(at 643.89 99.06 0)
+			(at 589.28 87.63 0)
 			(effects
 				(font

Commit message: Add platformIO
Parts:
- U14: value TCA9535PWR_C130204 -> TCA9535PWR
Changed lines of the file:
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@@
 			)
 		)
-		(property "Value" "TCA9535PWR_C130204"
+		(property "Value" "TCA9535PWR"
 			(at 556.26 163.83 0)
 			(effects

Commit message: Add battery ic
Parts:
- removed C24, C25: 1uF, Capacitor_SMD:C_1206_3216Metric, symbol Device:C_Small
- removed R100, R101, R102, R103, R99: 100R, symbol Device:R_Small
- removed R104, R105, R106, R107, R108, R98: 1k, symbol Device:R_Small
- removed R109, R110, R111, R112: 100k, symbol Device:R_Small
- removed R97: NCP18XH103F03RB, easyeda2kicad:R0603, symbol easyeda2kicad:NCP18XH103F03RB
- removed U14: TCA9535PWR, easyeda2kicad:TSSOP-24_L7.8-W4.4-P0.65-LS6.4-BL, symbol easyeda2kicad:TCA9535PWR_C130204
- removed U15: CD74HCT4051M96, easyeda2kicad:SOP-16_L10.0-W3.9-P1.27-LS6.0-BL, symbol easyeda2kicad:CD74HCT4051M96_C406862
- removed U7: MCP73833-AMI/MF, easyeda2kicad:DFN-10_L3.0-W3.0-P0.50-BL-EP-1, symbol easyeda2kicad:MCP73833-AMI_MF
- R113, R114, R117, R118: now not fitted
Connections:
- net GND: now also R115.1, R116.1, R117.1, R118.1
Other:
- added sheet Batteries Charging IC (Batteries_Charging_IC.kicad_sch)
